Commit message: tf & urdf fix

File: abb-packages/abb_irb120_support/urdf/irb120.urdf (robot description, URDF)
Before this commit: robot abb_irb120, 16 links, 15 joints
Joints:
- joint camera_view_joint: origin xyz=0.654 0.200 0.221 rpy=0 1.187 -3.142 -> xyz=0.06 0.11 0 rpy=0 0 0; parent camera_link -> base_link

File: abb-packages/abb_irb120_support/urdf/irb120_macro.xacro (robot description, xacro)
@@ -376,9 +376,15 @@
     </link>
      <joint name="camera_view_joint" type="fixed">
+        <origin xyz="0.06 0.11 0" rpy="0 0 0"/>
+      <parent link="base_link" />
+      <child link="camera_view_link"/>
+    </joint>
+    <link name="camera_view_link"/>
+     <!--joint name="camera_view_joint" type="fixed">
         <origin xyz="0.654 0.200 0.221" rpy="0 1.187 -3.142"/>
       <parent link="camera_link" />
       <child link="camera_view_link"/>
     </joint>
-    <link name="camera_view_link"/>
+    <link name="camera_view_link"/-->
   </xacro:macro>
 </robot>

Commit message: urdf

File: abb-packages/abb_irb120_support/urdf/irb120.urdf (robot description, URDF)
Before this commit: robot abb_irb120, 16 links, 15 joints
Links:
- added link left_gripper_link; visual box size=0.03 0.015 0.015
- added link right_gripper_link; visual box size=0.03 0.015 0.015
- link tool0: geometry visual box size=0.1 0.045 0.035
Joints:
- added joint left_gripper_joint: type prismatic, parent tool0, child left_gripper_link, origin xyz=0.0505 0 0 rpy=0 0 0, axis 0 1 0, limit lower=-0.02 upper=-0.01 effort=0 velocity=1
- added joint right_gripper_joint: type prismatic, parent tool0, child right_gripper_link, origin xyz=0.0505 0 0 rpy=0 0 0, axis 0 1 0, limit lower=-0.02 upper=-0.01 effort=0 velocity=1, mimic joint=left_gripper_joint multiplier=-1
- joint joint6-tool0: origin xyz=0 0 0 rpy=0 0 0 -> xyz=0.0505 0 0 rpy=0 0 0

File: abb-packages/abb_irb120_support/urdf/irb120_macro.xacro (robot description, xacro)
@@ -151,5 +151,33 @@
       </collision>
     </link>
-    <link name="${prefix}tool0"/>
+  <link name="${prefix}tool0">
+    <mass value="0.200"/>
+    <origin rpy="0 0 0" xyz="0 0 0"/>
+    <visual>
+      <origin rpy="0 0 0" xyz="0 0 0"/>
+      <geometry>
+        <box size="0.1 0.045 0.035"/>
+      </geometry>
+        <material name="orange"/>
+    </visual>
+  </link>
+<link name="${prefix}left_gripper_link">
+        <visual>
+            <geometry>
+                <box size="0.03 0.015 0.015" />
+            </geometry>
+        <material name="orange"/>
+        </visual>
+    </link>
+<link name="${prefix}right_gripper_link">
+        <visual>
+            <geometry>
+                <box size="0.03 0.015 0.015" />
+            </geometry>
+        <material name="orange">
+        <color rgba="0.1882353 0.1960784 0.2039216 1"/>
+      </material>
+        </visual>
+    </link>
     <!-- end of link list -->
     <!-- joint list -->
@@ -205,6 +233,21 @@
       <parent link="${prefix}link_6"/>
       <child link="${prefix}tool0"/>
-      <origin rpy="0 0 0" xyz="0 0 0"/>
-    </joint>
+    <origin rpy="0 0 0" xyz="0.0505 0 0"/>
+    </joint>
+  <joint name="${prefix}left_gripper_joint" type="prismatic">
+    <parent link="${prefix}tool0"/>
+    <child link="${prefix}left_gripper_link"/>
+    <axis xyz="0 1 0"/>
+    <limit lower="-0.02" upper="-0.01" effort="0" velocity="1" />
+    <origin rpy="0 0 0" xyz="0.0505 0 0"/>
+  </joint>
+  <joint name="${prefix}right_gripper_joint" type="prismatic">
+    <parent link="${prefix}tool0"/>
+    <child link="${prefix}right_gripper_link"/>
+    <axis xyz="0 1 0"/>
+    <limit lower="-0.02" upper="-0.01" effort="0" velocity="1" />
+    <origin rpy="0 0 0" xyz="0.0505 0 0"/>
+    <mimic joint="${prefix}left_gripper_joint" multiplier="-1" />
+  </joint>
     <!-- end of joint list -->
     <!-- ROS base_link to ABB World Coordinates transform -->

Commit message: urdf

File: abb-packages/abb_irb120_support/urdf/irb120.urdf (robot description, URDF)
Before this commit: robot abb_irb120, 18 links, 17 joints
Links:
- removed link left_gripper_link
- removed link right_gripper_link
- link tool0: geometry visual box size=0.155 0.005 0.005
Joints:
- removed joint left_gripper_joint
- removed joint right_gripper_joint
- joint joint6-tool0: origin xyz=0.0505 0 0 rpy=0 0 0 -> xyz=0.155 0 0 rpy=0 0 0

File: abb-packages/abb_irb120_support/urdf/irb120_macro.xacro (robot description, xacro)
@@ -152,15 +152,14 @@
     </link>
   <link name="${prefix}tool0">
-    <mass value="0.200"/>
     <origin rpy="0 0 0" xyz="0 0 0"/>
     <visual>
-      <origin rpy="0 0 0" xyz="0 0 0"/>
+      <origin rpy="0 0 0" xyz="-0.077 0 0"/>
       <geometry>
-        <box size="0.1 0.045 0.035"/>
+        <box size="0.155 0.005 0.005"/>
       </geometry>
         <material name="orange"/>
     </visual>
   </link>
-<link name="${prefix}left_gripper_link">
+<!--link name="${prefix}left_gripper_link">
         <visual>
             <geometry>
@@ -179,5 +178,5 @@
       </material>
         </visual>
-    </link>
+    </link-->
     <!-- end of link list -->
     <!-- joint list -->
@@ -233,7 +232,7 @@
       <parent link="${prefix}link_6"/>
       <child link="${prefix}tool0"/>
-    <origin rpy="0 0 0" xyz="0.0505 0 0"/>
-    </joint>
-  <joint name="${prefix}left_gripper_joint" type="prismatic">
+    <origin rpy="0 0 0" xyz="0.155 0 0"/>
+    </joint>
+  <!--joint name="${prefix}left_gripper_joint" type="prismatic">
     <parent link="${prefix}tool0"/>
     <child link="${prefix}left_gripper_link"/>
@@ -249,5 +248,5 @@
     <origin rpy="0 0 0" xyz="0.0505 0 0"/>
     <mimic joint="${prefix}left_gripper_joint" multiplier="-1" />
-  </joint>
+  </joint-->
     <!-- end of joint list -->
     <!-- ROS base_link to ABB World Coordinates transform -->

Commit message: urdf & path publisher

File: abb-packages/abb_irb120_support/urdf/irb120.urdf (robot description, URDF)
Before this commit: robot abb_irb120, 16 links, 15 joints
Links:
- link tool0: geometry collision box size=0.125 0.005 0.005; visual box size=0.125 0.005 0.005
Joints:
- joint joint6-tool0: origin xyz=0.155 0 0 rpy=0 0 0 -> xyz=0.125 0 0 rpy=0 0 0

File: abb-packages/abb_irb120_support/urdf/irb120_macro.xacro (robot description, xacro)
@@ -154,10 +154,16 @@
     <origin rpy="0 0 0" xyz="0 0 0"/>
     <visual>
-      <origin rpy="0 0 0" xyz="-0.077 0 0"/>
+      <origin rpy="0 0 0" xyz="-0.062 0 0"/>
       <geometry>
-        <box size="0.155 0.005 0.005"/>
+        <box size="0.125 0.005 0.005"/>
       </geometry>
         <material name="orange"/>
     </visual>
+    <collision>
+      <origin rpy="0 0 0" xyz="-0.062 0 0"/>
+      <geometry>
+        <box size="0.125 0.005 0.005"/>
+      </geometry>
+      </collision>
   </link>
 <!--link name="${prefix}left_gripper_link">
@@ -232,5 +238,5 @@
       <parent link="${prefix}link_6"/>
       <child link="${prefix}tool0"/>
-    <origin rpy="0 0 0" xyz="0.155 0 0"/>
+    <origin rpy="0 0 0" xyz="0.125 0 0"/>
     </joint>
   <!--joint name="${prefix}left_gripper_joint" type="prismatic">

Commit message: demo prep

File: abb-packages/abb_irb120_support/urdf/irb120.urdf (robot description, URDF)
Before this commit: robot abb_irb120, 16 links, 15 joints
Joints:
- joint camera_view_joint: origin xyz=0.06 0.11 0 rpy=0 0 0 -> xyz=0.069 0.1135 0 rpy=0 0 0
- joint joint_6: limit lower=-6.98132 upper=6.98132 effort=0 velocity=7.33038 -> lower=0 upper=6.98132 effort=0 velocity=7.33038

File: abb-packages/abb_irb120_support/urdf/irb120_macro.xacro (robot description, xacro)
@@ -231,5 +231,5 @@
       <parent link="${prefix}link_5"/>
       <child link="${prefix}link_6"/>
-      <limit effort="0" lower="-6.98132" upper="6.98132" velocity="7.33038"/>
+      <limit effort="0" lower="0" upper="6.98132" velocity="7.33038"/>
       <axis xyz="1 0 0"/>
       <dynamics damping="0.0" friction="0.0"/>
@@ -424,5 +424,5 @@
     </link>
      <joint name="camera_view_joint" type="fixed">
-        <origin xyz="0.06 0.11 0" rpy="0 0 0"/>
+        <origin xyz="0.069 0.1135 0" rpy="0 0 0"/>
       <parent link="base_link" />
       <child link="camera_view_link"/>

Commit message: Demo update and filtering

File: abb-packages/abb_irb120_support/urdf/irb120.urdf (robot description, URDF)
Before this commit: robot abb_irb120, 16 links, 15 joints
Joints:
- joint camera_view_joint: origin xyz=0.069 0.1135 0 rpy=0 0 0 -> xyz=0.0700 0.1130 0 rpy=0 0 0

File: abb-packages/abb_irb120_support/urdf/irb120_macro.xacro (robot description, xacro)
@@ -424,5 +424,5 @@
     </link>
      <joint name="camera_view_joint" type="fixed">
-        <origin xyz="0.069 0.1135 0" rpy="0 0 0"/>
+        <origin xyz="0.0700 0.1130 0" rpy="0 0 0"/>
       <parent link="base_link" />
       <child link="camera_view_link"/>

Commit message: update

File: abb-packages/abb_irb120_support/urdf/irb120.urdf (robot description, URDF)
Before this commit: robot abb_irb120, 16 links, 15 joints
Joints:
- joint camera_view_joint: origin xyz=0.0700 0.1130 0 rpy=0 0 0 -> xyz=0.0675 0.1155 0 rpy=0 0 0

File: abb-packages/abb_irb120_support/urdf/irb120_macro.xacro (robot description, xacro)
@@ -424,5 +424,5 @@
     </link>
      <joint name="camera_view_joint" type="fixed">
-        <origin xyz="0.0700 0.1130 0" rpy="0 0 0"/>
+        <origin xyz="0.0675 0.1155 0" rpy="0 0 0"/>
       <parent link="base_link" />
       <child link="camera_view_link"/>
